File: h9kx3.kicad_pcb (KiCad board)
At the start: 2 copper layers, 90 x 100 mm, 84 parts, among them CON1 AVR-ISP-6, J1 ACC1, J2 BAND, J3 ACC1_PC, J4 ACC2, J5 4BIT_BAND, J6 INH_IN, J7 KEYLINE_OUT, J8 PTT_POWERON_OUT, J9 CAN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

Commit message: pcb init
Parts:
- C1: value 47u -> 100n; footprint Capacitors_Tantalum_SMD:CP_Tantalum_Case-C_EIA-6032-28_Hand -> Capacitors_SMD:C_1206_HandSoldering
- moved Q3 123.9 mm to (272.3, 98.3)
- moved R16 112.7 mm to (260.8, 115.0)
- moved R29 107.8 mm to (253.8, 81.8)
- moved Q5 100.1 mm to (244.1, 75.3)
- moved R27 93.2 mm to (241.2, 95.5)
- moved R26 85.7 mm to (234.2, 102.1)
- moved Q7 83.5 mm to (231.8, 100.2)
- moved C1 80.8 mm to (228.3, 117.7)
- moved R28 78.8 mm to (227.1, 110.1)
- moved D4 76.1 mm to (204.0, 157.0), turned to 180 degrees
- moved R25 67.7 mm to (214.5, 120.0)
- moved D3 65.9 mm to (189.0, 157.0), turned to 180 degrees
- moved R23 60.0 mm to (192.1, 146.3), turned to 270 degrees
- moved R19 59.5 mm to (203.3, 81.7), turned to 90 degrees
- moved D2 57.9 mm to (174.0, 157.0), turned to 180 degrees
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Connections:
- net /RX renamed /RX_SCK
- C1 pad 1: +5V -> GND
- C1 pad 2: GND -> +5V
- J2 pad 1: Net-(J2-Pad1) -> +5V
- J2 pad 10: +5V -> Net-(J2-Pad10)
- J2 pad 11: Net-(J2-Pad11) -> +5V
- J2 pad 12: +5V -> Net-(J2-Pad12)
- J2 pad 13: Net-(J2-Pad13) -> +5V
- J2 pad 14: +5V -> Net-(J2-Pad14)
- J2 pad 15: Net-(J2-Pad15) -> +5V
- J2 pad 16: +5V -> Net-(J2-Pad16)
- J2 pad 17: Net-(J2-Pad17) -> +5V
- J2 pad 18: +5V -> Net-(J2-Pad18)
- J2 pad 19: Net-(J2-Pad19) -> +5V
- J2 pad 2: +5V -> Net-(J2-Pad2)
- J2 pad 20: +5V -> Net-(J2-Pad20)
- J2 pad 21: Net-(J2-Pad21) -> +5V
- J2 pad 22: +5V -> Net-(J2-Pad22)
- J2 pad 23: Net-(J2-Pad23) -> +5V
- J2 pad 24: +5V -> Net-(J2-Pad24)
- J2 pad 25: Net-(J2-Pad25) -> +5V
- J2 pad 26: +5V -> Net-(J2-Pad26)
- J2 pad 27: Net-(J2-Pad27) -> +5V
- J2 pad 28: +5V -> Net-(J2-Pad28)
- J2 pad 29: Net-(J2-Pad29) -> +5V
- J2 pad 3: Net-(J2-Pad3) -> +5V
- J2 pad 30: +5V -> Net-(J2-Pad30)
- J2 pad 31: Net-(J2-Pad31) -> +5V
- J2 pad 32: +5V -> Net-(J2-Pad32)
- J2 pad 4: +5V -> Net-(J2-Pad4)
- J2 pad 5: Net-(J2-Pad5) -> +5V
- J2 pad 6: +5V -> Net-(J2-Pad6)
- J2 pad 7: Net-(J2-Pad7) -> +5V
- J2 pad 8: +5V -> Net-(J2-Pad8)
- J2 pad 9: Net-(J2-Pad9) -> +5V
- R10 pad 2: Net-(J2-Pad15) -> Net-(J2-Pad16)
- R11 pad 2: Net-(J2-Pad17) -> Net-(J2-Pad18)
- R12 pad 2: Net-(J2-Pad19) -> Net-(J2-Pad20)
- R13 pad 2: Net-(J2-Pad21) -> Net-(J2-Pad22)
- R14 pad 2: Net-(J2-Pad23) -> Net-(J2-Pad24)
- R15 pad 2: Net-(J2-Pad25) -> Net-(J2-Pad26)
- R17 pad 2: Net-(J2-Pad27) -> Net-(J2-Pad28)
- R18 pad 2: Net-(J2-Pad29) -> Net-(J2-Pad30)
- R2 pad 2: Net-(J2-Pad1) -> Net-(J2-Pad2)
- R20 pad 2: Net-(J2-Pad31) -> Net-(J2-Pad32)
- R3 pad 2: Net-(J2-Pad3) -> Net-(J2-Pad4)
- R4 pad 2: Net-(J2-Pad5) -> Net-(J2-Pad6)
- R5 pad 2: Net-(J2-Pad7) -> Net-(J2-Pad8)
- R7 pad 2: Net-(J2-Pad9) -> Net-(J2-Pad10)
- R8 pad 2: Net-(J2-Pad11) -> Net-(J2-Pad12)
- R9 pad 2: Net-(J2-Pad13) -> Net-(J2-Pad14)
- U2 pad 13: (no net) -> /BAND_0
- U2 pad 14: (no net) -> /BAND_1
- U2 pad 15: (no net) -> /BAND_2
- U2 pad 16: /BAND_2 -> /BAND_3
- U2 pad 23: /BAND_3 -> (no net)
- U2 pad 8: /BAND_0 -> (no net)
- U2 pad 9: /BAND_1 -> (no net)
Routing:
- net +5V: track 0.00 -> 219.9 mm
- net VDD: track 0.00 -> 131.5 mm
- net /RX_SCK: track 0.00 -> 53.9 mm, vias 0 -> 1
- net /CAN_RX: track 0.00 -> 40.5 mm
- net Net-(R2-Pad1): track 0.00 -> 38.0 mm
- net /CAN_TX: track 0.00 -> 34.8 mm
- net Net-(J9-Pad0): track 0.00 -> 33.4 mm
- net Net-(R4-Pad1): track 0.00 -> 31.9 mm
- net Net-(J1-Pad3): track 0.00 -> 31.8 mm
- net Net-(C3-Pad1): track 0.00 -> 31.2 mm
- net /MISO: track 0.00 -> 28.2 mm
- net Net-(D7-Pad2): track 0.00 -> 27.8 mm
- net Net-(R3-Pad1): track 0.00 -> 27.4 mm
- net Net-(D6-Pad2): track 0.00 -> 27.3 mm
- net Net-(R7-Pad1): track 0.00 -> 27.2 mm
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- added copper zone on B.Cu, net GND
Other:
- net class Default: clearance 0.2 -> 0.25; trace_width 0.25 -> 0.4
- net class ISP added: clearance 0.25, trace_width 0.3, via_dia 0.6, via_drill 0.4
- net class PWR added: clearance 0.4, trace_width 0.5, via_dia 0.6, via_drill 0.4
- rule trace_clearance: 0.2 -> 0.25
- rule trace_min: 0.2 -> 0.3
- rule via_min_drill: 0.3 -> 0.4

Commit message: pcb
Parts:
- moved Q3 83.5 mm to (189.7, 85.6), turned to 180 degrees
- moved R16 70.6 mm to (190.6, 123.3), turned to 90 degrees
- moved R29 60.4 mm to (197.2, 102.9), turned to 270 degrees
- moved Q5 57.1 mm to (198.1, 109.1), turned to 270 degrees
- moved R27 54.4 mm to (194.6, 123.3), turned to 90 degrees
- moved R26 51.9 mm to (182.6, 95.9), turned to 90 degrees
- moved C1 46.3 mm to (183.9, 104.5), turned to 180 degrees
- moved R19 41.8 mm to (198.9, 123.3)
- moved Q7 39.1 mm to (196.5, 117.0), turned to 90 degrees
- moved R25 36.1 mm to (194.4, 89.9)
- moved R33 34.2 mm to (171.7, 88.4)
- moved R30 31.2 mm to (171.3, 82.2)
- moved Q6 28.0 mm to (165.0, 88.0), turned to 270 degrees
- moved R28 27.0 mm to (202.6, 98.8), turned to 180 degrees
- moved Q2 22.0 mm to (201.3, 115.4), turned to 180 degrees
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- renumbered CON1 to ISP
Connections:
- R21 pad 1: Net-(R21-Pad1) -> /LED_STATUS
- R22 pad 1: Net-(R22-Pad1) -> /LED_INH
- R23 pad 1: Net-(R23-Pad1) -> /LED_KEY
- U2 pad 18: Net-(R21-Pad1) -> (no net)
- U2 pad 22: Net-(R22-Pad1) -> /LED_STATUS
- U2 pad 23: (no net) -> /LED_INH
- U2 pad 24: (no net) -> /LED_KEY
- U2 pad 25: Net-(R23-Pad1) -> /INHIBITS
- U2 pad 27: /KX3_POWER_ON -> /PTT_OUT
- U2 pad 28: /PTT_OUT -> /KX3_POWER_ON
- U2 pad 3: /INHIBITS -> (no net)
- U3 pad None: (no net) -> GND
Routing:
- net +5V: track 219.9 -> 275.4 mm
- net Net-(C5-Pad1): track 0.00 -> 53.2 mm
- net /INHIBITS: track 0.00 -> 51.7 mm
- net Net-(C16-Pad1): track 3.93 -> 48.2 mm
- net Net-(C17-Pad1): track 3.93 -> 41.4 mm
- net Net-(Q6-Pad1): track 0.00 -> 29.9 mm
- net /KEYLINE: track 0.00 -> 29.9 mm
- net Net-(D4-Pad2): track 0.00 -> 29.3 mm
- net /INHIBITS_IN: track 0.00 -> 28.8 mm
- net Net-(D2-Pad2): track 0.00 -> 28.0 mm
- net GND: track 18.9 -> 43.8 mm, vias 4 -> 32
- net Net-(D3-Pad2): track 0.00 -> 24.6 mm
- net Net-(C7-Pad1): track 16.6 -> 40.7 mm
- net Net-(C6-Pad1): track 0.00 -> 20.6 mm
- net /LED_KEY: track 0.00 -> 14.8 mm
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Other:
- board text added: "SQ8KFH"
- board text added: "h9kx3 band decoder v1"

Commit message: fix
Parts:
- added ?: , kfhlib:VIA, F.Cu at (138.0, 120.0)
- added ?: , kfhlib:VIA, F.Cu at (136.0, 116.0)
- added ?: , kfhlib:VIA, F.Cu at (134.0, 116.0)
- added ?: , kfhlib:VIA, F.Cu at (132.0, 116.0)
- added ?: , kfhlib:VIA, F.Cu at (138.0, 114.0)
- added ?: , kfhlib:VIA, F.Cu at (136.0, 114.0)
- added ?: , kfhlib:VIA, F.Cu at (134.0, 114.0)
- added ?: , kfhlib:VIA, F.Cu at (132.0, 114.0)
- added ?: , kfhlib:VIA, F.Cu at (136.0, 120.0)
- added ?: , kfhlib:VIA, F.Cu at (134.0, 120.0)
- added ?: , kfhlib:VIA, F.Cu at (132.0, 120.0)
- added ?: , kfhlib:VIA, F.Cu at (138.0, 118.0)
- added ?: , kfhlib:VIA, F.Cu at (136.0, 118.0)
- added ?: , kfhlib:VIA, F.Cu at (134.0, 118.0)
- added ?: , kfhlib:VIA, F.Cu at (132.0, 118.0)
- added ?: , kfhlib:VIA, F.Cu at (138.0, 116.0)
Routing:
- net GND: vias 32 -> 31
Other:
- board text added: "h9kx3 band decoder v1.0"
- board text removed: "h9kx3 band decoder v1"
Changed lines of the file:
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@@
 (kicad_pcb (version 4) (host pcbnew 4.0.6)
   (general
-    (links 198)
+    (links 214)
     (no_connects 0)
-    (area 119.924999 61.924999 210.075001 162.075001)
+    (area 119.924999 55.084999 222.564286 162.100001)
     (thickness 1.6)
     (drawings 10)
-    (tracks 537)
+    (tracks 535)
     (zones 0)
-    (modules 84)
+    (modules 100)
     (nets 81)
   )
@@
     (title "h9kx3 band decoder")
     (date 2019-05-09)
-    (rev 1)
+    (rev 1.0)
     (company SQ8KFH)
   )
@@
   )
   (setup
-    (last_trace_width 0.5)
+    (last_trace_width 0.4)
     (user_trace_width 0.3)
     (user_trace_width 0.4)
@@
     (mod_text_size 1 1)
     (mod_text_width 0.15)
-    (pad_size 4.5 4.5)
-    (pad_drill 3.5)
+    (pad_size 0.6 0.6)
+    (pad_drill 0.4)
     (pad_to_mask_clearance 0.2)
     (aux_axis_origin 0 0)
     (visible_elements FFFFFF7F)
     (pcbplotparams
-      (layerselection 0x00030_80000001)
-      (usegerberextensions false)
+      (layerselection 0x010e0_80000001)
+      (usegerberextensions true)
       (excludeedgelayer true)
       (linewidth 0.100000)
@@
       (outputformat 1)
       (mirror false)
-      (drillshape 1)
+      (drillshape 0)
       (scaleselection 1)
-      (outputdirectory ""))
+      (outputdirectory gerber/))
   )
   (net 0 "")
@@
     (add_net VDD)
   )
+  (module kfhlib:VIA (layer F.Cu)
+    (at 137.953 120.046)
+    (tags VIA)
+    (fp_text reference "" (at 0.1 2.2) (layer F.Fab) hide
+      (effects (font (size 1 1) (thickness 0.15)))
+    )
+    (fp_text value "" (at -0.05 -2) (layer F.Fab) hide
+      (effects (font (size 1 1) (thickness 0.15)))
+    )
+    (pad 1 thru_hole circle (at 0 0) (size 0.6 0.6) (drill 0.4) (layers *.Cu)
+      (net 2 GND) (zone_connect 2))
+  )
+  (module kfhlib:VIA (layer F.Cu)
+    (at 135.953 120.046)
+    (tags VIA)
+    (fp_text reference "" (at 0.1 2.2) (layer F.Fab) hide
+      (effects (font (size 1 1) (thickness 0.15)))
+    )
+    (fp_text value "" (at -0.05 -2) (layer F.Fab) hide
+      (effects (font (size 1 1) (thickness 0.15)))
+    )
+    (pad 1 thru_hole circle (at 0 0) (size 0.6 0.6) (drill 0.4) (layers *.Cu)
+      (net 2 GND) (zone_connect 2))
+  )
+  (module kfhlib:VIA (layer F.Cu)
+    (at 133.953 120.046)
+    (tags VIA)
+    (fp_text reference "" (at 0.1 2.2) (layer F.Fab) hide
+      (effects (font (size 1 1) (thickness 0.15)))
+    )
+    (fp_text value "" (at -0.05 -2) (layer F.Fab) hide
+      (effects (font (size 1 1) (thickness 0.15)))
+    )
+    (pad 1 thru_hole circle (at 0 0) (size 0.6 0.6) (drill 0.4) (layers *.Cu)
+      (net 2 GND) (zone_connect 2))
+  )
+  (module kfhlib:VIA (layer F.Cu)
+    (at 131.953 120.046)
+    (tags VIA)
+    (fp_text reference "" (at 0.1 2.2) (layer F.Fab) hide
+      (effects (font (size 1 1) (thickness 0.15)))
+    )
+    (fp_text value "" (at -0.05 -2) (layer F.Fab) hide
+      (effects (font (size 1 1) (thickness 0.15)))
+    )
+    (pad 1 thru_hole circle (at 0 0) (size 0.6 0.6) (drill 0.4) (layers *.Cu)
+      (net 2 GND) (zone_connect 2))
+  )
+  (module kfhlib:VIA (layer F.Cu)
+    (at 137.953 118.046)
+    (tags VIA)
+    (fp_text reference "" (at 0.1 2.2) (layer F.Fab) hide
+      (effects (font (size 1 1) (thickness 0.15)))
+    )
+    (fp_text value "" (at -0.05 -2) (layer F.Fab) hide
+      (effects (font (size 1 1) (thickness 0.15)))
+    )
+    (pad 1 thru_hole circle (at 0 0) (size 0.6 0.6) (drill 0.4) (layers *.Cu)
+      (net 2 GND) (zone_connect 2))
+  )
+  (module kfhlib:VIA (layer F.Cu)
+    (at 135.953 118.046)
+    (tags VIA)
+    (fp_text reference "" (at 0.1 2.2) (layer F.Fab) hide
+      (effects (font (size 1 1) (thickness 0.15)))
+    )
+    (fp_text value "" (at -0.05 -2) (layer F.Fab) hide
+      (effects (font (size 1 1) (thickness 0.15)))
+    )
+    (pad 1 thru_hole circle (at 0 0) (size 0.6 0.6) (drill 0.4) (layers *.Cu)
+      (net 2 GND) (zone_connect 2))
+  )
+  (module kfhlib:VIA (layer F.Cu)
+    (at 133.953 118.046)
+    (tags VIA)
+    (fp_text reference "" (at 0.1 2.2) (layer F.Fab) hide
+      (effects (font (size 1 1) (thickness 0.15)))
+    )
+    (fp_text value "" (at -0.05 -2) (layer F.Fab) hide
+      (effects (font (size 1 1) (thickness 0.15)))
+    )
+    (pad 1 thru_hole circle (at 0 0) (size 0.6 0.6) (drill 0.4) (layers *.Cu)
+      (net 2 GND) (zone_connect 2))
+  )
+  (module kfhlib:VIA (layer F.Cu)
+    (at 131.953 118.046)
+    (tags VIA)
+    (fp_text reference "" (at 0.1 2.2) (layer F.Fab) hide
+      (effects (font (size 1 1) (thickness 0.15)))
+    )
+    (fp_text value "" (at -0.05 -2) (layer F.Fab) hide
+      (effects (font (size 1 1) (thickness 0.15)))
+    )
+    (pad 1 thru_hole circle (at 0 0) (size 0.6 0.6) (drill 0.4) (layers *.Cu)
+      (net 2 GND) (zone_connect 2))
+  )
+  (module kfhlib:VIA (layer F.Cu)
+    (at 137.953 116.046)
+    (tags VIA)
+    (fp_text reference "" (at 0.1 2.2) (layer F.Fab) hide
+      (effects (font (size 1 1) (thickness 0.15)))
+    )
+    (fp_text value "" (at -0.05 -2) (layer F.Fab) hide
+      (effects (font (size 1 1) (thickness 0.15)))
+    )
+    (pad 1 thru_hole circle (at 0 0) (size 0.6 0.6) (drill 0.4) (layers *.Cu)
+      (net 2 GND) (zone_connect 2))
+  )
+  (module kfhlib:VIA (layer F.Cu)
+    (at 135.953 116.046)
+    (tags VIA)
+    (fp_text reference "" (at 0.1 2.2) (layer F.Fab) hide
+      (effects (font (size 1 1) (thickness 0.15)))
+    )
+    (fp_text value "" (at -0.05 -2) (layer F.Fab) hide
+      (effects (font (size 1 1) (thickness 0.15)))
+    )
+    (pad 1 thru_hole circle (at 0 0) (size 0.6 0.6) (drill 0.4) (layers *.Cu)
+      (net 2 GND) (zone_connect 2))
+  )
+  (module kfhlib:VIA (layer F.Cu)
+    (at 133.953 116.046)
+    (tags VIA)
+    (fp_text reference "" (at 0.1 2.2) (layer F.Fab) hide
+      (effects (font (size 1 1) (thickness 0.15)))
+    )
+    (fp_text value "" (at -0.05 -2) (layer F.Fab) hide
+      (effects (font (size 1 1) (thickness 0.15)))
+    )
+    (pad 1 thru_hole circle (at 0 0) (size 0.6 0.6) (drill 0.4) (layers *.Cu)
+      (net 2 GND) (zone_connect 2))
+  )
+  (module kfhlib:VIA (layer F.Cu)
+    (at 131.953 116.046)
+    (tags VIA)
+    (fp_text reference "" (at 0.1 2.2) (layer F.Fab) hide
+      (effects (font (size 1 1) (thickness 0.15)))
+    )
+    (fp_text value "" (at -0.05 -2) (layer F.Fab) hide
+      (effects (font (size 1 1) (thickness 0.15)))
+    )
+    (pad 1 thru_hole circle (at 0 0) (size 0.6 0.6) (drill 0.4) (layers *.Cu)
+      (net 2 GND) (zone_connect 2))
+  )
+  (module kfhlib:VIA (layer F.Cu)
+    (at 137.953 114.046)
+    (tags VIA)
+    (fp_text reference "" (at 0.1 2.2) (layer F.Fab) hide
+      (effects (font (size 1 1) (thickness 0.15)))
+    )
+    (fp_text value "" (at -0.05 -2) (layer F.Fab) hide
+      (effects (font (size 1 1) (thickness 0.15)))
+    )
+    (pad 1 thru_hole circle (at 0 0) (size 0.6 0.6) (drill 0.4) (layers *.Cu)
+      (net 2 GND) (zone_connect 2))
+  )
+  (module kfhlib:VIA (layer F.Cu)
+    (at 135.953 114.046)
+    (tags VIA)
+    (fp_text reference "" (at 0.1 2.2) (layer F.Fab) hide
+      (effects (font (size 1 1) (thickness 0.15)))
+    )
+    (fp_text value "" (at -0.05 -2) (layer F.Fab) hide
+      (effects (font (size 1 1) (thickness 0.15)))
+    )
+    (pad 1 thru_hole circle (at 0 0) (size 0.6 0.6) (drill 0.4) (layers *.Cu)
+      (net 2 GND) (zone_connect 2))
+  )
+  (module kfhlib:VIA (layer F.Cu)
+    (at 133.953 114.046)
+    (tags VIA)
+    (fp_text reference "" (at 0.1 2.2) (layer F.Fab) hide
+      (effects (font (size 1 1) (thickness 0.15)))
+    )
+    (fp_text value "" (at -0.05 -2) (layer F.Fab) hide
+      (effects (font (size 1 1) (thickness 0.15)))
+    )
+    (pad 1 thru_hole circle (at 0 0) (size 0.6 0.6) (drill 0.4) (layers *.Cu)
+      (net 2 GND) (zone_connect 2))
+  )
   (module Capacitors_SMD:C_1206_HandSoldering (layer F.Cu)
     (at 157.338 111.708)
@@
     )
   )
+  (module kfhlib:VIA (layer F.Cu)
+    (at 131.953 114.046)
+    (tags VIA)
+    (fp_text reference "" (at 0.1 2.2) (layer F.Fab) hide
+      (effects (font (size 1 1) (thickness 0.15)))
+    )
+    (fp_text value "" (at -0.05 -2) (layer F.Fab) hide
+      (effects (font (size 1 1) (thickness 0.15)))
+    )
+    (pad 1 thru_hole circle (at 0 0) (size 0.6 0.6) (drill 0.4) (layers *.Cu)
+      (net 2 GND) (zone_connect 2))
+  )
   (gr_text SQ8KFH (at 197.1675 139.6365) (layer F.Cu)
     (effects (font (size 1.6 1.6) (thickness 0.3)))
   )
-  (gr_text "h9kx3 band decoder v1" (at 146.7485 157.861) (layer F.SilkS)
+  (gr_text "h9kx3 band decoder v1.0\n" (at 146.7485 157.861) (layer F.SilkS)
     (effects (font (size 2 2) (thickness 0.4)))
   )
@@
   (segment (start 125.068 125.932) (end 125 126) (width 0.4) (layer B.Cu) (net 2))
   (via (at 125 126) (size 0.6) (drill 0.4) (layers F.Cu B.Cu) (net 2))
-  (via (at 134.989 117.042) (size 0.6) (drill 0.4) (layers F.Cu B.Cu) (net 2))
-  (segment (start 134.989 117.042) (end 134.986 117.042) (width 0.4) (layer B.Cu) (net 2))
   (via (at 125.839 117.042) (size 0.6) (drill 0.4) (layers F.Cu B.Cu) (net 2))
   (segment (start 125.839 117.042) (end 125.842 117.042) (width 0.4) (layer B.Cu) (net 2))
